File: pre_amp.brd (EAGLE design)
At the start: 100 x 80 mm, 51 parts, among them Q1 BF245, Q2 BF245, Q3 BF245

Commit message: [#1] PCB layout
Parts:
- C2: device resistor:E3,5-8 -> resistor:E5-8,5
- R5: device resistor:0204/7 -> resistor:0207/10
- moved R17 189.1 mm to (91.4, 17.8), turned to 90 degrees
- moved Q3 187.1 mm to (86.4, 16.5)
- moved R16 171.1 mm to (81.3, 17.8), turned to 90 degrees
- moved MUTE_1 165.9 mm to (64.8, 14.0), turned to 270 degrees
- moved R15 163.6 mm to (86.4, 24.1)
- moved C10 162.4 mm to (86.4, 29.2), turned to 180 degrees
- moved ULTRA_HIGH_1 157.7 mm to (66.0, 31.8)
- moved OUT_GND 154.6 mm to (90.2, 38.1)
- moved R7 150.8 mm to (52.1, 21.6), turned to 90 degrees
- moved R13 150.4 mm to (74.9, 14.0), turned to 180 degrees
- moved Q2 147.7 mm to (61.0, 27.9), turned to 180 degrees
- moved BASS_CUT2 135.3 mm to (35.6, 14.0), turned to 180 degrees
- moved C6 134.9 mm to (61.0, 20.3), turned to 270 degrees
- moved C9 131.4 mm to (74.9, 21.6), turned to 90 degrees
- moved OUT_P 130.2 mm to (82.5, 38.1)
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Connections:
- net GND: now also R5.2; no longer R5.1
- net N$4: now also R5.1; no longer R5.2
Routing:
- net GND: track 0.00 -> 278.2 mm, vias 0 -> 2
- net VCC: track 0.00 -> 124.2 mm
- net N$14: track 0.00 -> 40.7 mm
- net N$15: track 0.00 -> 37.0 mm
- net N$4: track 0.00 -> 29.0 mm
- net N$9: track 0.00 -> 25.0 mm
- net N$3: track 0.00 -> 17.9 mm
- net N$18: track 0.00 -> 17.3 mm
- net N$16: track 0.00 -> 17.0 mm
- net N$7: track 0.00 -> 16.4 mm
- net N$19: track 0.00 -> 15.5 mm
- net N$10: track 0.00 -> 13.3 mm
- net N$8: track 0.00 -> 12.0 mm
- net N$20: track 0.00 -> 10.9 mm
- net N$13: track 0.00 -> 10.3 mm
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Other:
- board size 100 x 80 mm -> 98.7 x 44.4 mm
